File: main.sch (EAGLE design)
At the start: 25 parts, among them IC1 STM32F030F4P, IC3 ACS712, J1 22-05-7028-02, J2 22-27-2051-05, Q1 8MHz, Q2 BC639, Q3 BC640, Q4 IRF540, SW1 EC12E_SW, U1 MAX485CSA+

Commit message: lay2
Parts:
- removed IC3: ACS712, ACS712:ACS712
- removed R6: 1K, resistor:R-EU_R1206
- removed R7: 1K5, resistor:R-EU_R1206
Connections:
- removed net N$19: IC3.I-_0, J1-1.S
- removed net N$20: IC3.VOUT, R6.2
- removed net N$21: IC1MCU.PA1, R6.1, R7.2
- removed net N$7: IC1MCU.NRST, J2-2.S, R1.2
- new net N$22: IC1MCU.NRST, R1.2
- net +5V: no longer IC3.VCC
- net GND: no longer IC3.GND, R7.1
- net N$16: now also J1-1.S; no longer IC3.I+_1
Changed lines of the file:
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@@
 <setting verticaltext="up"/>
 </settings>
-<grid distance="0.1" unitdist="inch" unit="inch" style="lines" multiple="1" display="yes" altdistance="0.01" altunitdist="inch" altunit="inch"/>
+<grid distance="0.1" unitdist="inch" unit="inch" style="lines" multiple="1" display="no" altdistance="0.01" altunitdist="inch" altunit="inch"/>
 <layers>
 <layer number="1" name="Top" color="4" fill="1" visible="no" active="no"/>
@@
 <part name="P+8" library="supply1" deviceset="VCC" device=""/>
 <part name="J2" library="con-molex" deviceset="22-?-05" device="27-2051"/>
-<part name="IC3" library="ACS712" deviceset="ACS712" device=""/>
-<part name="P+10" library="supply1" deviceset="+5V" device=""/>
-<part name="R6" library="resistor" deviceset="R-EU_" device="R1206" value="1K"/>
-<part name="R7" library="resistor" deviceset="R-EU_" device="R1206" value="1K5"/>
-<part name="GND9" library="supply1" deviceset="GND" device=""/>
-<part name="GND10" library="supply1" deviceset="GND" device=""/>
 </parts>
 <sheets>
@@
 <attribute name="NAME" x="50.8" y="97.282" size="1.524" layer="95" rot="R180"/>
 </instance>
-<instance part="J2" gate="-2" x="53.34" y="93.98" rot="R180"/>
 <instance part="J2" gate="-3" x="53.34" y="91.44" rot="R180"/>
 <instance part="J2" gate="-4" x="53.34" y="88.9" rot="R180"/>
 <instance part="J2" gate="-5" x="53.34" y="86.36" rot="R180"/>
-<instance part="IC3" gate="A" x="182.88" y="132.08"/>
-<instance part="P+10" gate="1" x="200.66" y="144.78"/>
-<instance part="R6" gate="G$1" x="208.28" y="106.68" smashed="yes" rot="R90">
-<attribute name="NAME" x="206.7814" y="102.87" size="1.778" layer="95" rot="R90"/>
-<attribute name="VALUE" x="211.582" y="102.87" size="1.778" layer="96" rot="R90"/>
-</instance>
-<instance part="R7" gate="G$1" x="208.28" y="91.44" smashed="yes" rot="R90">
-<attribute name="NAME" x="206.7814" y="87.63" size="1.778" layer="95" rot="R90"/>
-<attribute name="VALUE" x="211.582" y="87.63" size="1.778" layer="96" rot="R90"/>
-</instance>
-<instance part="GND9" gate="1" x="208.28" y="81.28"/>
-<instance part="GND10" gate="1" x="200.66" y="121.92"/>
 </instances>
 <busses>
@@
 <pinref part="J2" gate="-5" pin="S"/>
 </segment>
-<segment>
-<pinref part="R7" gate="G$1" pin="1"/>
-<wire x1="208.28" y1="86.36" x2="208.28" y2="83.82" width="0.1524" layer="91"/>
-<pinref part="GND9" gate="1" pin="GND"/>
-</segment>
-<segment>
-<pinref part="IC3" gate="A" pin="GND"/>
-<pinref part="GND10" gate="1" pin="GND"/>
-<wire x1="198.12" y1="127" x2="200.66" y2="127" width="0.1524" layer="91"/>
-<wire x1="200.66" y1="127" x2="200.66" y2="124.46" width="0.1524" layer="91"/>
-</segment>
-</net>
-<net name="N$7" class="0">
-<segment>
-<pinref part="IC1" gate="MCU" pin="NRST"/>
-<wire x1="27.94" y1="45.72" x2="25.4" y2="45.72" width="0.1524" layer="91"/>
-<pinref part="R1" gate="G$1" pin="2"/>
-<wire x1="25.4" y1="45.72" x2="22.86" y2="45.72" width="0.1524" layer="91"/>
-<wire x1="25.4" y1="45.72" x2="25.4" y2="63.5" width="0.1524" layer="91"/>
-<wire x1="25.4" y1="63.5" x2="30.48" y2="63.5" width="0.1524" layer="91"/>
-<wire x1="30.48" y1="63.5" x2="30.48" y2="93.98" width="0.1524" layer="91"/>
-<pinref part="J2" gate="-2" pin="S"/>
-<wire x1="30.48" y1="93.98" x2="55.88" y2="93.98" width="0.1524" layer="91"/>
-<junction x="25.4" y="45.72"/>
-</segment>
 </net>
 <net name="N$6" class="0">
@@
 <wire x1="30.48" y1="15.24" x2="30.48" y2="17.78" width="0.1524" layer="91"/>
 </segment>
-<segment>
-<pinref part="IC3" gate="A" pin="VCC"/>
-<wire x1="198.12" y1="137.16" x2="200.66" y2="137.16" width="0.1524" layer="91"/>
-<pinref part="P+10" gate="1" pin="+5V"/>
-<wire x1="200.66" y1="137.16" x2="200.66" y2="142.24" width="0.1524" layer="91"/>
-</segment>
 </net>
 <net name="N$17" class="0">
@@
 <segment>
 <pinref part="F1" gate="1" pin="2"/>
-<pinref part="IC3" gate="A" pin="I+_1"/>
 <wire x1="139.7" y1="134.62" x2="167.64" y2="134.62" width="0.1524" layer="91"/>
-</segment>
-</net>
-<net name="N$19" class="0">
-<segment>
-<pinref part="IC3" gate="A" pin="I-_0"/>
 <wire x1="167.64" y1="129.54" x2="162.56" y2="129.54" width="0.1524" layer="91"/>
 <pinref part="J1" gate="-1" pin="S"/>
-</segment>
-</net>
-<net name="N$20" class="0">
-<segment>
-<pinref part="IC3" gate="A" pin="VOUT"/>
-<wire x1="208.28" y1="134.62" x2="198.12" y2="134.62" width="0.1524" layer="91"/>
-<pinref part="R6" gate="G$1" pin="2"/>
-<wire x1="208.28" y1="134.62" x2="208.28" y2="111.76" width="0.1524" layer="91"/>
-</segment>
-</net>
-<net name="N$21" class="0">
-<segment>
-<pinref part="R6" gate="G$1" pin="1"/>
-<pinref part="R7" gate="G$1" pin="2"/>
-<wire x1="208.28" y1="101.6" x2="208.28" y2="99.06" width="0.1524" layer="91"/>
-<pinref part="IC1" gate="MCU" pin="PA1"/>
-<wire x1="208.28" y1="99.06" x2="208.28" y2="96.52" width="0.1524" layer="91"/>
-<wire x1="73.66" y1="45.72" x2="162.56" y2="45.72" width="0.1524" layer="91"/>
-<wire x1="162.56" y1="45.72" x2="162.56" y2="99.06" width="0.1524" layer="91"/>
-<wire x1="162.56" y1="99.06" x2="208.28" y2="99.06" width="0.1524" layer="91"/>
-<junction x="208.28" y="99.06"/>
-</segment>
-</net>
+<wire x1="167.64" y1="134.62" x2="167.64" y2="129.54" width="0.1524" layer="91"/>
+</segment>
+</net>
+<net name="N$22" class="0">
+<segment>
+<pinref part="R1" gate="G$1" pin="2"/>
+<pinref part="IC1" gate="MCU" pin="NRST"/>
+<wire x1="27.94" y1="45.72" x2="22.86" y2="45.72" width="0.1524" layer="91"/>
+</segment>
+</net>
